File: plantbright.kicad_sch (KiCad schematic)
At the start: 23 parts, among them J1 POWER OUT, J2 USB-C, Q1 AO3400A, Q2 AO3400A, Q3 AO3400A, Q5 AO3400A, SW1 USER 0, U1 XIAO-ESP32-C6

Commit message: Add cap
Parts:
- added C1: 100uF, Capacitor_THT:CP_Radial_D5.0mm_P2.50mm, symbol Device:C_Polarized
Connections:
- net +5V: now also C1.1
- net GND: now also C1.2
Changed lines of the file:
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@@
 	(rectangle
 		(start 17.78 17.78)
-		(end 190.5 96.52)
+		(end 196.85 96.52)
 		(stroke
 			(width 0)
@@
 	(text "POWER"
 		(exclude_from_sim no)
-		(at 104.14 94.996 0)
+		(at 107.188 94.742 0)
 		(effects
 			(font
@@
 	)
 	(junction
+		(at 184.15 36.83)
+		(diameter 0)
+		(color 0 0 0 0)
+	)
+	(junction
 		(at 82.55 73.66)
 		(diameter 0)
@@
 	(wire
 		(pts
+			(xy 184.15 36.83) (xy 184.15 49.53)
+		)
+		(stroke
+			(width 0)
+			(type default)
+		)
+	)
+	(wire
+		(pts
 			(xy 73.66 116.84) (xy 73.66 119.38)
 		)
@@
 	(wire
 		(pts
-			(xy 157.48 36.83) (xy 172.72 36.83)
+			(xy 157.48 36.83) (xy 184.15 36.83)
 		)
 		(stroke
@@
 	(wire
 		(pts
-			(xy 172.72 36.83) (xy 172.72 31.75)
+			(xy 184.15 36.83) (xy 184.15 31.75)
 		)
 		(stroke
@@
 	(wire
 		(pts
+			(xy 184.15 57.15) (xy 184.15 63.5)
+		)
+		(stroke
+			(width 0)
+			(type default)
+		)
+	)
+	(wire
+		(pts
 			(xy 40.64 35.56) (xy 43.18 35.56)
 		)
@@
 	)
 	(symbol
+		(lib_id "Device:C_Polarized")
+		(at 184.15 53.34 0)
+		(unit 1)
+		(exclude_from_sim no)
+		(in_bom yes)
+		(on_board yes)
+		(dnp no)
+		(fields_autoplaced yes)
+		(property "Reference" "C1"
+			(at 187.96 51.1809 0)
+			(effects
+				(font
+					(size 1.27 1.27)
+				)
+				(justify left)
+			)
+		)
+		(property "Value" "100uF"
+			(at 187.96 53.7209 0)
+			(effects
+				(font
+					(size 1.27 1.27)
+				)
+				(justify left)
+			)
+		)
+		(property "Footprint" "Capacitor_THT:CP_Radial_D5.0mm_P2.50mm"
+			(at 185.1152 57.15 0)
+			(effects
+				(font
+					(size 1.27 1.27)
+				)
+				(hide yes)
+			)
+		)
+		(property "Datasheet" "~"
+			(at 184.15 53.34 0)
+			(effects
+				(font
+					(size 1.27 1.27)
+				)
+				(hide yes)
+			)
+		)
+		(property "Description" "Polarized capacitor"
+			(at 184.15 53.34 0)
+			(effects
+				(font
+					(size 1.27 1.27)
+				)
+				(hide yes)
+			)
+		)
+		(pin "2"
+		)
+		(pin "1"
+		)
+		(instances
+			(project ""
+				(path "/e2caaa62-12a4-4d86-8d92-9420077836ea"
+					(reference "C1")
+					(unit 1)
+				)
+			)
+		)
+	)
+	(symbol
 		(lib_id "Connector:Screw_Terminal_01x05")
 		(at 44.45 120.65 0)
@@
 	(symbol
 		(lib_id "power:+5V")
-		(at 172.72 31.75 0)
+		(at 184.15 31.75 0)
 		(unit 1)
 		(exclude_from_sim no)
@@
 		(fields_autoplaced yes)
 		(property "Reference" "#PWR020"
-			(at 172.72 35.56 0)
+			(at 184.15 35.56 0)
 			(effects
 				(font
@@
 		)
 		(property "Value" "+5V"
-			(at 172.72 26.67 0)
+			(at 184.15 26.67 0)
 			(effects
 				(font
@@
 		)
 		(property "Footprint" ""
-			(at 172.72 31.75 0)
+			(at 184.15 31.75 0)
 			(effects
 				(font
@@
 		)
 		(property "Datasheet" ""
-			(at 172.72 31.75 0)
+			(at 184.15 31.75 0)
 			(effects
 				(font
@@
 		)
 		(property "Description" "Power symbol creates a global label with name \"+5V\""
-			(at 172.72 31.75 0)
+			(at 184.15 31.75 0)
 			(effects
 				(font
@@
 					(unit 1)
 				)
+			)
+		)
+	)
+	(symbol
+		(lib_id "power:GND")
+		(at 184.15 63.5 0)
+		(unit 1)
+		(exclude_from_sim no)
+		(in_bom yes)
+		(on_board yes)
+		(dnp no)
+		(fields_autoplaced yes)
+		(property "Reference" "#PWR017"
+			(at 184.15 69.85 0)
+			(effects
+				(font
+					(size 1.27 1.27)
+				)
+				(hide yes)
+			)
+		)
+		(property "Value" "GND"
+			(at 184.15 68.58 0)
+			(effects
+				(font
+					(size 1.27 1.27)
+				)
+			)
+		)
+		(property "Footprint" ""
+			(at 184.15 63.5 0)
+			(effects
+				(font
+					(size 1.27 1.27)
+				)
+				(hide yes)
+			)
+		)
+		(property "Datasheet" ""
+			(at 184.15 63.5 0)
+			(effects
+				(font
+					(size 1.27 1.27)
+				)
+				(hide yes)
+			)
+		)
+		(property "Description" "Power symbol creates a global label with name \"GND\" , ground"
+			(at 184.15 63.5 0)
+			(effects
+				(font
+					(size 1.27 1.27)
+				)
+				(hide yes)
+			)
+		)
+		(pin "1"
+		)
+		(instances
+			(project "plantbright"
+				(path "/e2caaa62-12a4-4d86-8d92-9420077836ea"
+					(reference "#PWR017")
+					(unit 1)
+				)

Commit message: Ground pour
Connections:
- net at J1.2 (Pin_2): now also R13.2; no longer R10.2
- net at J1.3 (Pin_3): now also R12.2; no longer R11.2
- net at J1.4 (Pin_4): now also R11.2; no longer R12.2
- net at J1.5 (Pin_5): now also R10.2; no longer R13.2
Other:
- moved on the sheet: R10, R11, R12, R13

Commit message: DRC, getting there.
Parts:
- C1: footprint Capacitor_THT:CP_Radial_D5.0mm_P2.50mm -> Capacitor_SMD:C_1206_3216Metric_Pad1.33x1.80mm_HandSolder
Changed lines of the file:
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@@
 			)
 		)
-		(property "Footprint" "Capacitor_THT:CP_Radial_D5.0mm_P2.50mm"
+		(property "Footprint" "Capacitor_SMD:C_1206_3216Metric_Pad1.33x1.80mm_HandSolder"
 			(at 185.1152 57.15 0)
 			(effects

Commit message: Yay, V1.
Connections:
- net BTN_1: now also U1.3 (GPIO2/A2/D2); no longer U1.5 (GPIO22/D4/SDA)
- net CH_3: now also U1.10 (GPIO20/D9/MISO); no longer U1.3 (GPIO2/A2/D2)
- net CH_4: now also U1.11 (GPIO18/D10/MOSI); no longer U1.4 (GPIO21/D3)
